Commit message: URDF description + visualization

File: src/robotics_toolbox/robots/robot_hw.urdf (robot description, URDF)
Before this commit: robot simple_robot, 2 links, 1 joints
Links:
- added link link_0_cylinder; visual cylinder length=0.5 radius=0.05
- added link link_1_sphere; visual sphere radius=0.06
- added link link_2_cylinder; visual cylinder length=0.25 radius=0.05
- added link link_3_cylinder; visual cylinder length=0.25 radius=0.05
- added link link_4_sphere; visual sphere radius=0.06
- added link link_5_cylinder; visual cylinder length=0.25 radius=0.05
- link base_link: geometry visual box size=0.3 0.3 0.3
Joints:
- added joint joint1: type fixed, parent link_0_cylinder, child link_1_sphere, origin xyz=0 0 0.5 rpy=0 0 0
- added joint joint2: type revolute, parent link_1_sphere, child link_2_cylinder, origin xyz=0 0 0 rpy=0 0 0, axis 1 0 0, limit lower=-1.5707963267948966 upper=1.5707963267948966 effort=1000.0 velocity=0.5
- added joint joint3: type revolute, parent link_2_cylinder, child link_3_cylinder, origin xyz=0 0 0.25 rpy=0 0 0, axis 0 0 1, limit lower=-1.5707963267948966 upper=1.5707963267948966 effort=1000.0 velocity=0.5
- added joint joint4: type fixed, parent link_3_cylinder, child link_4_sphere, origin xyz=0 0 0.25 rpy=0 0 0
- added joint joint5: type revolute, parent link_4_sphere, child link_5_cylinder, origin xyz=0 0 0 rpy=0 0 0, axis 1 0 0, limit lower=-1.5707963267948966 upper=1.5707963267948966 effort=1000.0 velocity=0.5
- added joint joint6: type fixed, parent link_5_cylinder, child end_effector, origin xyz=0 0 0.25 rpy=0 0 0
- joint joint0: axis (none) -> 0 0 1; child end_effector -> link_0_cylinder; limit (none) -> lower=-1.5707963267948966 upper=1.5707963267948966 effort=1000.0 velocity=0.5; origin xyz=0 0 0 rpy=0 0 0 -> xyz=0 0 0.15 rpy=0 0 0; type fixed -> revolute
